File: pcb/ScartPCB.kicad_pcb (KiCad board)
At the start: 4 copper layers, 39.5 x 21 mm, 13 parts, among them J1 Conn_02x10_Odd_Even, J2 R, J3 G, J4 B, J5 SYNC, J6 AUD, J7 GND

Commit message: Revising PCB
Parts:
- added LOGO1: OSHW-Logo2_7.3x6mm_SilkScreen, Symbol:OSHW-Logo2_7.3x6mm_SilkScreen, B.Cu at (136.1, 115.2)
Other:
- board text added: "AUD"
- board text added: "AUDIO"
- board text added: "B"
- board text added: "BLUE"
- board text added: "G"
- board text added: "GND"
- board text added: "GREEN"
- board text added: "P2000T SCART"
- board text added: "R"
- board text added: "RED"
- board text added: "SYNC"
- board text added: "rev1"
